Commit message: omega клешня

File: urdf/ebobot.urdf (robot description, URDF)
Before this commit: robot turtlebro, 6 links, 5 joints
Links:
- added link arm; visual box size=0.1 0.05 0.05
- added link arm_box; visual box size=0.05 0.05 0.05
Joints:
- added joint arm_box_joint: type fixed, parent base_link, child arm_box, origin xyz=0.08 0.08 0.1 rpy=0 0 0.785
- added joint arm_joint: type revolute, parent arm_box, child arm, origin xyz=0.0 0.0 0.0 rpy=0 0 0.0, axis 0 1 0, limit lower=1.57 upper=-1.28 effort=1.0 velocity=0.01

Commit message: urdf baza

File: urdf/ebobot.urdf (robot description, URDF)
Before this commit: robot ebobot, 8 links, 7 joints
Links:
- added link baza; visual cylinder length=0.01 radius=0.16
Joints:
- added joint baza_joint: type fixed, parent base_footprint, child baza, origin xyz=0.0 0.0 0.0 rpy=0.0 0.0 0.0
